File: megawing/soundpuddle_megawing_mk2.brd (EAGLE design)
At the start: 149.2 x 123.8 mm, 363 parts, among them J1 POWER_JACKPTH, Q1 MOSFET-P_CHANNELDPACK, Q2 MOSFET-P_CHANNELDPACK, SW1 SPST_TACT-EVQQ2, SW2 ROTARY_ENCODER_SW_2CH_LED2XXS, SW3 ROTARY_ENCODER_SW_2CH_LED2XXS, T1 COMMON_MODE_CHOKEBIG_FOOT, U1 LTC3854, U10 SN74HCT541DW, U11 SN74HCT541DW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

Commit message: updated eagle files for the MK2 PCB. Some component values are not yet final, hardware is in initial physical testing phase
Parts:
- R10, R9: value 1K -> 100K
- R106: value 100K -> 1M
- R5: value 1K -> DNP
Connections:
- net N$283 renamed CH7_CLK
- net N$284 renamed CH7_DATA
- net N$285 renamed CH6_CLK
- net N$287 renamed CH5_CLK
- net N$297 renamed CH3_DATA
- net N$298 renamed CH3_CLK
- net N$299 renamed CH2_CLK
- net N$300 renamed CH2_DATA
- net N$301 renamed CH1_CLK
- net N$302 renamed CH1_DATA
- net N$346 renamed CH11_CLK
- net N$347 renamed CH11_DATA
- net N$348 renamed CH10_DATA
- net N$349 renamed CH10_CLK
- net N$350 renamed CH9_DATA
- net N$351 renamed CH8_CLK
- net N$366 renamed CH8_DATA
- net N$367 renamed CH4_CLK
- net N$368 renamed CH4_DATA
- net N$369 renamed CH12_CLK
- net N$370 renamed CH12_DATA
- net N$373 renamed CH9_CLK
- removed net N$286: JP14.2, R37.P$6
- removed net N$288: JP11.2, R37.P$8
- new net CH5_DATA: JP11.2, JP14.2, R37.P$6, R37.P$8
Routing:
- net CH5_DATA: track 0.00 -> 21.2 mm
- net N$288: track 12.3 -> 0.00 mm
- net N$286: track 8.96 -> 0.00 mm
Changed lines of the file:
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@@
 <layer number="14" name="Route14" color="1" fill="6" visible="no" active="no"/>
 <layer number="15" name="PWR" color="11" fill="1" visible="no" active="yes"/>
-<layer number="16" name="Bottom" color="1" fill="1" visible="yes" active="yes"/>
+<layer number="16" name="Bottom" color="1" fill="1" visible="no" active="yes"/>
 <layer number="17" name="Pads" color="2" fill="1" visible="yes" active="yes"/>
 <layer number="18" name="Vias" color="2" fill="1" visible="yes" active="yes"/>
@@
 <attribute name="VALUE" x="-52.0845" y="-16.975" size="0.762" layer="27"/>
 </element>
-<element name="R106" library="1_Dan Master" package="0603" value="100K" x="-55.3085" y="-13.2715" smashed="yes">
+<element name="R106" library="1_Dan Master" package="0603" value="1M" x="-55.3085" y="-13.2715" smashed="yes">
 <attribute name="NAME" x="-56.3925" y="-12.6325" size="0.889" layer="25" font="vector"/>
 <attribute name="VALUE" x="-56.1485" y="-14.435" size="0.762" layer="27"/>
@@
 <attribute name="VALUE" x="1.22" y="37.7135" size="0.762" layer="27" rot="R180"/>
 </element>
-<element name="R10" library="1_Dan Master" package="0603" value="1K" x="7.5565" y="44.1325" smashed="yes">
+<element name="R10" library="1_Dan Master" package="0603" value="100K" x="7.5565" y="44.1325" smashed="yes">
 <attribute name="NAME" x="8.853" y="43.7233" size="1.016" layer="25" font="vector"/>
 <attribute name="VALUE" x="6.273" y="42.6775" size="0.762" layer="27"/>
 </element>
-<element name="R9" library="1_Dan Master" package="0603" value="1K" x="4.2545" y="44.1325" smashed="yes" rot="R180">
+<element name="R9" library="1_Dan Master" package="0603" value="100K" x="4.2545" y="44.1325" smashed="yes" rot="R180">
 <attribute name="NAME" x="1.487" y="43.7233" size="1.016" layer="25" font="vector"/>
 <attribute name="VALUE" x="5.538" y="45.5875" size="0.762" layer="27" rot="R180"/>
@@
 <attribute name="VALUE" x="5.538" y="42.0315" size="0.762" layer="27" rot="R180"/>
 </element>
-<element name="R5" library="1_Dan Master" package="0603" value="1K" x="-0.0635" y="42.8625" smashed="yes">
+<element name="R5" library="1_Dan Master" package="0603" value="DNP" x="-0.0635" y="42.8625" smashed="yes">
 <attribute name="NAME" x="-2.958" y="42.3263" size="1.016" layer="25" font="vector"/>
 <attribute name="VALUE" x="-1.347" y="41.4075" size="0.762" layer="27"/>
@@
 <wire x1="50.3555" y1="-21.6535" x2="52.5845" y2="-19.4245" width="0.381" layer="1"/>
 </signal>
-<signal name="N$283">
+<signal name="CH7_CLK">
 <contactref element="R41" pad="P$8"/>
 <contactref element="JP17" pad="3"/>
@@
 <wire x1="65.0875" y1="-17.2085" x2="65.0875" y2="-18.7325" width="0.381" layer="1"/>
 </signal>
-<signal name="N$284">
+<signal name="CH7_DATA">
 <contactref element="R41" pad="P$7"/>
 <contactref element="JP17" pad="2"/>
@@
 <wire x1="62.5475" y1="-17.4625" x2="62.5475" y2="-18.7325" width="0.381" layer="1"/>
 </signal>
-<signal name="N$285">
+<signal name="CH6_CLK">
 <contactref element="R37" pad="P$5"/>
 <contactref element="JP14" pad="3"/>
@@
 <wire x1="65.0875" y1="-12.3825" x2="65.0875" y2="-14.2875" width="0.381" layer="1"/>
 </signal>
-<signal name="N$286">
-<contactref element="R37" pad="P$6"/>
-<contactref element="JP14" pad="2"/>
-<wire x1="55.3945" y1="-14.0525" x2="58.7565" y2="-14.0525" width="0.381" layer="1"/>
-<wire x1="58.7565" y1="-14.0525" x2="59.1185" y2="-14.4145" width="0.381" layer="1"/>
-<wire x1="59.1185" y1="-14.4145" x2="61.9125" y2="-14.4145" width="0.381" layer="1"/>
-<wire x1="61.9125" y1="-14.4145" x2="62.5475" y2="-13.7795" width="0.381" layer="1"/>
-<wire x1="62.5475" y1="-12.3825" x2="62.5475" y2="-13.7795" width="0.381" layer="1"/>
-</signal>
-<signal name="N$287">
+<signal name="CH5_CLK">
 <contactref element="JP11" pad="3"/>
 <contactref element="R37" pad="P$7"/>
@@
 <wire x1="65.0875" y1="-6.0325" x2="65.0875" y2="-7.6835" width="0.381" layer="1"/>
 </signal>
-<signal name="N$288">
+<signal name="CH5_DATA">
 <contactref element="JP11" pad="2"/>
 <contactref element="R37" pad="P$8"/>
@@
 <wire x1="61.9125" y1="-8.0645" x2="62.5475" y2="-7.4295" width="0.381" layer="1"/>
 <wire x1="62.5475" y1="-6.0325" x2="62.5475" y2="-7.4295" width="0.381" layer="1"/>
+<contactref element="R37" pad="P$6"/>
+<contactref element="JP14" pad="2"/>
+<wire x1="55.3945" y1="-14.0525" x2="58.7565" y2="-14.0525" width="0.381" layer="1"/>
+<wire x1="58.7565" y1="-14.0525" x2="59.1185" y2="-14.4145" width="0.381" layer="1"/>
+<wire x1="59.1185" y1="-14.4145" x2="61.9125" y2="-14.4145" width="0.381" layer="1"/>
+<wire x1="61.9125" y1="-14.4145" x2="62.5475" y2="-13.7795" width="0.381" layer="1"/>
+<wire x1="62.5475" y1="-12.3825" x2="62.5475" y2="-13.7795" width="0.381" layer="1"/>
+<wire x1="55.3945" y1="-14.0525" x2="55.3945" y2="-12.4525" width="0" layer="19" extent="1-1"/>
 </signal>
 <signal name="N$289">
@@
 <wire x1="49.2135" y1="0.4445" x2="50.3555" y2="0.4445" width="0.381" layer="1"/>
 </signal>
-<signal name="N$297">
+<signal name="CH3_DATA">
 <contactref element="R39" pad="P$8"/>
 <contactref element="JP16" pad="2"/>
@@
 <wire x1="62.5475" y1="6.6675" x2="62.5475" y2="5.5245" width="0.381" layer="1"/>
 </signal>
-<signal name="N$298">
+<signal name="CH3_CLK">
 <contactref element="R39" pad="P$7"/>
 <contactref element="JP16" pad="3"/>
@@
 <wire x1="65.0875" y1="6.6675" x2="65.0875" y2="4.7625" width="0.381" layer="1"/>
 </signal>
-<signal name="N$299">
+<signal name="CH2_CLK">
 <contactref element="R36" pad="P$5"/>
 <contactref element="JP13" pad="3"/>
@@
 <wire x1="65.0875" y1="13.0175" x2="65.0875" y2="11.3665" width="0.381" layer="1"/>
 </signal>
-<signal name="N$300">
+<signal name="CH2_DATA">
 <contactref element="R36" pad="P$6"/>
 <contactref element="JP13" pad="2"/>
@@
 <wire x1="62.5475" y1="13.0175" x2="62.5475" y2="11.8745" width="0.381" layer="1"/>
 </signal>
-<signal name="N$301">
+<signal name="CH1_CLK">
 <contactref element="JP10" pad="3"/>
 <contactref element="R36" pad="P$7"/>
@@
 <wire x1="65.0875" y1="19.3675" x2="65.0875" y2="17.9705" width="0.381" layer="1"/>
 </signal>
-<signal name="N$302">
+<signal name="CH1_DATA">
 <contactref element="JP10" pad="2"/>
 <contactref element="R36" pad="P$8"/>
@@
 <wire x1="53.4445" y1="-40.7605" x2="52.3305" y2="-40.7605" width="0.381" layer="1"/>
 </signal>
-<signal name="N$346">
+<signal name="CH11_CLK">
 <contactref element="R43" pad="P$8"/>
 <contactref element="JP18" pad="3"/>
@@
 <wire x1="65.0875" y1="-42.3545" x2="65.0875" y2="-44.1325" width="0.381" layer="1"/>
 </signal>
-<signal name="N$347">
+<signal name="CH11_DATA">
 <contactref element="R43" pad="P$7"/>
 <contactref element="JP18" pad="2"/>
@@
 <wire x1="62.5475" y1="-42.3545" x2="62.5475" y2="-44.1325" width="0.381" layer="1"/>
 </signal>
-<signal name="N$348">
+<signal name="CH10_DATA">
 <contactref element="R38" pad="P$5"/>
 <contactref element="JP15" pad="2"/>
@@
 <wire x1="62.5475" y1="-36.5125" x2="62.5475" y2="-37.7825" width="0.381" layer="1"/>
 </signal>
-<signal name="N$349">
+<signal name="CH10_CLK">
 <contactref element="R38" pad="P$6"/>
 <contactref element="JP15" pad="3"/>
@@
 <wire x1="65.0875" y1="-36.2585" x2="65.0875" y2="-37.7825" width="0.381" layer="1"/>
 </signal>
-<signal name="N$350">
+<signal name="CH9_DATA">
 <contactref element="R38" pad="P$8"/>
 <wire x1="55.3945" y1="-33.2805" x2="61.8425" y2="-33.2805" width="0.381" layer="1"/>
@@
 <wire x1="62.5475" y1="-32.5755" x2="62.5475" y2="-31.4325" width="0.381" layer="1"/>
 </signal>
-<signal name="N$351">
+<signal name="CH8_CLK">
 <contactref element="R41" pad="P$6"/>
 <contactref element="JP20" pad="3"/>
@@
 <wire x1="65.0875" y1="-23.8125" x2="65.0875" y2="-25.0825" width="0.381" layer="1"/>
 </signal>
-<signal name="N$366">
+<signal name="CH8_DATA">
 <contactref element="R41" pad="P$5"/>
 <contactref element="JP20" pad="2"/>
@@
 <wire x1="62.5475" y1="-23.8125" x2="62.5475" y2="-25.0825" width="0.381" layer="1"/>
 </signal>
-<signal name="N$367">
+<signal name="CH4_CLK">
 <contactref element="R39" pad="P$6"/>
 <contactref element="JP19" pad="3"/>
@@
 <wire x1="65.0875" y1="2.6655" x2="65.0875" y2="0.3175" width="0.381" layer="1"/>
 </signal>
-<signal name="N$368">
+<signal name="CH4_DATA">
 <contactref element="R39" pad="P$5"/>
 <contactref element="JP19" pad="2"/>
@@
 <wire x1="62.5475" y1="1.8415" x2="62.5475" y2="0.3175" width="0.381" layer="1"/>
 </signal>
-<signal name="N$369">
+<signal name="CH12_CLK">
 <contactref element="R43" pad="P$6"/>
 <contactref element="JP21" pad="3"/>
@@
 <wire x1="65.0875" y1="-50.4825" x2="65.0875" y2="-52.9575" width="0.381" layer="1"/>
 </signal>
-<signal name="N$370">
+<signal name="CH12_DATA">
 <contactref element="R43" pad="P$5"/>
 <contactref element="JP21" pad="2"/>
@@
 <wire x1="62.5475" y1="-52.9575" x2="62.5475" y2="-50.4825" width="0.381" layer="1"/>
 </signal>
-<signal name="N$373">
+<signal name="CH9_CLK">
 <contactref element="R38" pad="P$7"/>
 <wire x1="55.3945" y1="-34.0805" x2="64.0905" y2="-34.0805" width="0.381" layer="1"/>
@@
 </signal>
 </signals>
-<errors>
-</errors>
 </board>
 </drawing>
