File: megawing/soundpuddle_megawing_mk2.sch (EAGLE design)
At the start: 362 parts, among them J1 POWER_JACKPTH, Q1 MOSFET-P_CHANNELDPACK, Q2 MOSFET-P_CHANNELDPACK, SW1 SPST_TACT-EVQQ2, SW2 ROTARY_ENCODER_SW_2CH_LED2XXS, SW3 ROTARY_ENCODER_SW_2CH_LED2XXS, T1 COMMON_MODE_CHOKEBIG_FOOT, U1 LTC3854, U10 SN74HCT541DW, U11 SN74HCT541DW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

Commit message: updated eagle files for the MK2 PCB. Some component values are not yet final, hardware is in initial physical testing phase
Parts:
- R10, R9: value 1K -> 100K
- R106: value 100K -> 1M
- R5: value 1K -> DNP
Connections:
- net N$283 renamed CH7_CLK
- net N$284 renamed CH7_DATA
- net N$285 renamed CH6_CLK
- net N$287 renamed CH5_CLK
- net N$297 renamed CH3_DATA
- net N$298 renamed CH3_CLK
- net N$299 renamed CH2_CLK
- net N$300 renamed CH2_DATA
- net N$301 renamed CH1_CLK
- net N$302 renamed CH1_DATA
- net N$346 renamed CH11_CLK
- net N$347 renamed CH11_DATA
- net N$348 renamed CH10_DATA
- net N$349 renamed CH10_CLK
- net N$350 renamed CH9_DATA
- net N$351 renamed CH8_CLK
- net N$366 renamed CH8_DATA
- net N$367 renamed CH4_CLK
- net N$368 renamed CH4_DATA
- net N$369 renamed CH12_CLK
- net N$370 renamed CH12_DATA
- net N$373 renamed CH9_CLK
- removed net N$286: JP14.2, R37.3.2
- removed net N$288: JP11.2, R37.1.2
- new net CH5_DATA: JP11.2, JP14.2, R37.1.2, R37.3.2
Other:
- note added: "FIX THESE VALUES"
- note removed: "Confirm the Sync pin"
- note removed: "FIX THESE PINS"
Changed lines of the file:
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@@
 <part name="C147" library="1_Dan Master" deviceset="CAPACITOR" device="C_0603" value="1uF"/>
 <part name="C135" library="1_Dan Master" deviceset="CAPACITOR" device="C_0603" value="1uF"/>
-<part name="R106" library="1_Dan Master" deviceset="RESISTOR" device="R_0603" value="100K"/>
+<part name="R106" library="1_Dan Master" deviceset="RESISTOR" device="R_0603" value="1M"/>
 <part name="C132" library="1_Dan Master" deviceset="CAPACITOR" device="C_0603" value="100pF"/>
 <part name="GND35" library="supply1" deviceset="GNDA" device=""/>
@@
 <part name="U2" library="1_Dan Master" deviceset="LTC2955" device="TS8"/>
 <part name="C39" library="1_Dan Master" deviceset="CAPACITOR" device="C_0603" value="0.1uF"/>
-<part name="R10" library="1_Dan Master" deviceset="RESISTOR" device="R_0603" value="1K"/>
-<part name="R9" library="1_Dan Master" deviceset="RESISTOR" device="R_0603" value="1K"/>
+<part name="R10" library="1_Dan Master" deviceset="RESISTOR" device="R_0603" value="100K"/>
+<part name="R9" library="1_Dan Master" deviceset="RESISTOR" device="R_0603" value="100K"/>
 <part name="R8" library="1_Dan Master" deviceset="RESISTOR" device="R_0603" value="DNP"/>
 <part name="R7" library="1_Dan Master" deviceset="RESISTOR" device="R_0603" value="100K"/>
@@
 <part name="JP4" library="1_Dan Master" deviceset="HEADER-SMALL-1PIN" device=""/>
 <part name="R6" library="1_Dan Master" deviceset="RESISTOR" device="R_0603" value="1K"/>
-<part name="R5" library="1_Dan Master" deviceset="RESISTOR" device="R_0603" value="1K"/>
+<part name="R5" library="1_Dan Master" deviceset="RESISTOR" device="R_0603" value="DNP"/>
 <part name="R19" library="1_Dan Master" deviceset="RESISTOR" device="R_0603" value="1K"/>
 <part name="C4" library="1_Dan Master" deviceset="CAPACITOR" device="C_1206" value="10uF"/>
@@
 <plain>
 <text x="-452.12" y="-144.78" size="7.62" layer="97">Bluetooth</text>
-<text x="-25.4" y="101.6" size="5.08" layer="97">Confirm the Sync pin</text>
 <text x="-447.04" y="-292.1" size="7.62" layer="97">MIDI Input</text>
-<text x="-25.4" y="172.72" size="6.4516" layer="97">FIX THESE PINS</text>
+<text x="-314.96" y="177.8" size="6.4516" layer="97">FIX THESE VALUES</text>
 <text x="-81.28" y="-147.32" size="1.778" layer="97">*This reset line needs to be actively controlled</text>
 <text x="-149.86" y="-208.28" size="1.778" layer="97">Place R164 to enable BT secondary PCM input</text>
@@
 <instance part="U4" gate="C_POWER" x="-325.12" y="111.76"/>
 <instance part="U4" gate="G$1" x="-238.76" y="132.08"/>
-<instance part="U4" gate="G$2" x="-238.76" y="104.14"/>
+<instance part="U4" gate="G$2" x="-238.76" y="96.52"/>
 <instance part="U4" gate="G$3" x="-322.58" y="50.8"/>
 <instance part="U4" gate="G$4" x="-386.08" y="50.8"/>
@@
 <pinref part="C56" gate="G$1" pin="2"/>
 <wire x1="-264.16" y1="96.52" x2="-264.16" y2="93.98" width="0.1524" layer="91"/>
-<wire x1="-264.16" y1="93.98" x2="-256.54" y2="93.98" width="0.1524" layer="91"/>
-<wire x1="-256.54" y1="93.98" x2="-256.54" y2="101.6" width="0.1524" layer="91"/>
 <pinref part="U4" gate="G$2" pin="GND"/>
-<wire x1="-256.54" y1="101.6" x2="-248.92" y2="101.6" width="0.1524" layer="91"/>
+<wire x1="-264.16" y1="93.98" x2="-248.92" y2="93.98" width="0.1524" layer="91"/>
 <wire x1="-264.16" y1="93.98" x2="-264.16" y2="91.44" width="0.1524" layer="91"/>
 <pinref part="GND8" gate="1" pin="GND"/>
@@
 </segment>
 </net>
-<net name="N$283" class="0">
+<net name="CH7_CLK" class="0">
 <segment>
 <wire x1="-58.42" y1="-40.64" x2="-17.78" y2="-40.64" width="0.1524" layer="91"/>
@@
 </segment>
 </net>
-<net name="N$284" class="0">
+<net name="CH7_DATA" class="0">
 <segment>
 <wire x1="-20.32" y1="-43.18" x2="-48.26" y2="-43.18" width="0.1524" layer="91"/>
@@
 </segment>
 </net>
-<net name="N$285" class="0">
+<net name="CH6_CLK" class="0">
 <segment>
 <wire x1="15.24" y1="-60.96" x2="10.16" y2="-60.96" width="0.1524" layer="91"/>
@@
 </segment>
 </net>
-<net name="N$286" class="0">
-<segment>
-<wire x1="-12.7" y1="-35.56" x2="-38.1" y2="-35.56" width="0.1524" layer="91"/>
-<wire x1="-12.7" y1="-35.56" x2="-12.7" y2="-60.96" width="0.1524" layer="91"/>
-<pinref part="R37" gate=".3" pin="2"/>
-<wire x1="15.24" y1="-63.5" x2="10.16" y2="-63.5" width="0.1524" layer="91"/>
-<wire x1="10.16" y1="-63.5" x2="7.62" y2="-60.96" width="0.1524" layer="91"/>
-<wire x1="7.62" y1="-60.96" x2="-12.7" y2="-60.96" width="0.1524" layer="91"/>
-<pinref part="JP14" gate="G$1" pin="2"/>
-</segment>
-</net>
-<net name="N$287" class="0">
+<net name="CH5_CLK" class="0">
 <segment>
 <wire x1="-48.26" y1="-33.02" x2="-10.16" y2="-33.02" width="0.1524" layer="91"/>
@@
 </segment>
 </net>
-<net name="N$288" class="0">
+<net name="CH5_DATA" class="0">
 <segment>
 <wire x1="-7.62" y1="-30.48" x2="-58.42" y2="-30.48" width="0.1524" layer="91"/>
@@
 <pinref part="R37" gate=".1" pin="2"/>
 </segment>
+<segment>
+<wire x1="-12.7" y1="-35.56" x2="-38.1" y2="-35.56" width="0.1524" layer="91"/>
+<wire x1="-12.7" y1="-35.56" x2="-12.7" y2="-60.96" width="0.1524" layer="91"/>
+<pinref part="R37" gate=".3" pin="2"/>
+<wire x1="15.24" y1="-63.5" x2="10.16" y2="-63.5" width="0.1524" layer="91"/>
+<wire x1="10.16" y1="-63.5" x2="7.62" y2="-60.96" width="0.1524" layer="91"/>
+<wire x1="7.62" y1="-60.96" x2="-12.7" y2="-60.96" width="0.1524" layer="91"/>
+<pinref part="JP14" gate="G$1" pin="2"/>
+</segment>
 </net>
 <net name="N$289" class="0">
@@
 </segment>
 </net>
-<net name="N$297" class="0">
+<net name="CH3_DATA" class="0">
 <segment>
 <wire x1="-309.88" y1="-40.64" x2="-269.24" y2="-40.64" width="0.1524" layer="91"/>
@@
 </segment>
 </net>
-<net name="N$298" class="0">
+<net name="CH3_CLK" class="0">
 <segment>
 <wire x1="-271.78" y1="-43.18" x2="-299.72" y2="-43.18" width="0.1524" layer="91"/>
@@
 </segment>
 </net>
-<net name="N$299" class="0">
+<net name="CH2_CLK" class="0">
 <segment>
 <wire x1="-279.4" y1="-38.1" x2="-266.7" y2="-38.1" width="0.1524" layer="91"/>
@@
 </segment>
 </net>
-<net name="N$300" class="0">
+<net name="CH2_DATA" class="0">
 <segment>
 <wire x1="-264.16" y1="-35.56" x2="-289.56" y2="-35.56" width="0.1524" layer="91"/>
@@
 </segment>
 </net>
-<net name="N$301" class="0">
+<net name="CH1_CLK" class="0">
 <segment>
 <wire x1="-299.72" y1="-33.02" x2="-261.62" y2="-33.02" width="0.1524" layer="91"/>
@@
 </segment>
 </net>
-<net name="N$302" class="0">
+<net name="CH1_DATA" class="0">
 <segment>
 <wire x1="-259.08" y1="-30.48" x2="-309.88" y2="-30.48" width="0.1524" layer="91"/>
@@
 </segment>
 </net>
-<net name="N$346" class="0">
+<net name="CH11_CLK" class="0">
 <segment>
 <wire x1="231.14" y1="-40.64" x2="271.78" y2="-40.64" width="0.1524" layer="91"/>
@@
 </segment>
 </net>
-<net name="N$347" class="0">
+<net name="CH11_DATA" class="0">
 <segment>
 <wire x1="269.24" y1="-43.18" x2="241.3" y2="-43.18" width="0.1524" layer="91"/>
@@
 </segment>
 </net>
-<net name="N$348" class="0">
+<net name="CH10_DATA" class="0">
 <segment>
 <wire x1="261.62" y1="-38.1" x2="274.32" y2="-38.1" width="0.1524" layer="91"/>
@@
 </segment>
 </net>
-<net name="N$349" class="0">
+<net name="CH10_CLK" class="0">
 <segment>
 <wire x1="276.86" y1="-35.56" x2="251.46" y2="-35.56" width="0.1524" layer="91"/>
@@
 </segment>
 </net>
-<net name="N$350" class="0">
+<net name="CH9_DATA" class="0">
 <segment>
 <wire x1="281.94" y1="-30.48" x2="231.14" y2="-30.48" width="0.1524" layer="91"/>
@@
 </segment>
 </net>
-<net name="N$351" class="0">
+<net name="CH8_CLK" class="0">
 <segment>
 <wire x1="15.24" y1="-106.68" x2="-22.86" y2="-106.68" width="0.1524" layer="91"/>
@@
 </segment>
 </net>
-<net name="N$366" class="0">
+<net name="CH8_DATA" class="0">
 <segment>
 <wire x1="15.24" y1="-109.22" x2="-25.4" y2="-109.22" width="0.1524" layer="91"/>
@@
 </segment>
 </net>
-<net name="N$367" class="0">
+<net name="CH4_CLK" class="0">
 <segment>
 <wire x1="-236.22" y1="-106.68" x2="-274.32" y2="-106.68" width="0.1524" layer="91"/>
@@
 </segment>
 </net>
-<net name="N$368" class="0">
+<net name="CH4_DATA" class="0">
 <segment>
 <wire x1="-279.4" y1="-48.26" x2="-276.86" y2="-48.26" width="0.1524" layer="91"/>
@@
 </segment>
 </net>
-<net name="N$369" class="0">
+<net name="CH12_CLK" class="0">
 <segment>
 <wire x1="266.7" y1="-106.68" x2="266.7" y2="-45.72" width="0.1524" layer="91"/>
@@
 </segment>
 </net>
-<net name="N$370" class="0">
+<net name="CH12_DATA" class="0">
 <segment>
 <wire x1="261.62" y1="-48.26" x2="264.16" y2="-48.26" width="0.1524" layer="91"/>
@@
 </segment>
 </net>
-<net name="N$373" class="0">
+<net name="CH9_CLK" class="0">
 <segment>
 <wire x1="241.3" y1="-33.02" x2="279.4" y2="-33.02" width="0.1524" layer="91"/>
@@
 <pinref part="C56" gate="G$1" pin="1"/>
 <wire x1="-264.16" y1="104.14" x2="-264.16" y2="106.68" width="0.1524" layer="91"/>
-<wire x1="-248.92" y1="106.68" x2="-264.16" y2="106.68" width="0.1524" layer="91"/>
+<wire x1="-248.92" y1="99.06" x2="-254" y2="99.06" width="0.1524" layer="91"/>
+<wire x1="-254" y1="99.06" x2="-254" y2="106.68" width="0.1524" layer="91"/>
+<wire x1="-254" y1="106.68" x2="-264.16" y2="106.68" width="0.1524" layer="91"/>
 <pinref part="FB5" gate="G$1" pin="2"/>
 <wire x1="-264.16" y1="109.22" x2="-264.16" y2="106.68" width="0.1524" layer="91"/>
